Commit message: Add wheel to chassis

File: midge_ws/src/midge/urdf/midge.xacro (robot description, xacro)
@@ -1,4 +1,20 @@
 <?xml version='1.0'?>
 <robot name="midge" xmlns:xacro="http://www.ros.org/wiki/xacro">
+  <joint type="continuous" name="left_wheel_hinge">
+    <origin xyz="0 0.30 0" rpy="0 0 0" />
+    <parent link="chassis"/>
+    <child link="left_wheel" />
+    <axis xyz="0 1 0" rpy="0 0 0" />
+    <limit effort="10000" velocity="1000" />
+    <dynamics damping="1.0" friction="1.0" />
+  </joint>
+  <joint type="continuous" name="right_wheel_hinge">
+    <origin xyz="0 -0.30 0" rpy="0 0 0" />
+    <parent link="chassis"/>
+    <child link="right_wheel" />
+    <axis xyz="0 1 0" rpy="0 0 0" />
+    <limit effort="10000" velocity="1000" />
+    <dynamics damping="1.0" friction="1.0" />
+  </joint>
   <link name='chassis'>
     <pose>0 0 0.1 0 0 0</pose>
@@ -49,3 +65,49 @@
     </visual>
   </link>
+  <link name="left_wheel">
+    <inertial>
+      <mass value="5"/>
+      <origin xyz="0 0 0" rpy="0 1.5707 1.5707"/>
+      <inertia
+        ixx="0.1" ixy="0.0" ixz="0.0"
+        iyy="0.1" iyz="0.0"
+        izz="0.1"
+      />
+    </inertial>
+    <collision>
+      <origin xyz="0 0 0" rpy="0 1.5707 1.5707"/>
+      <geometry>
+        <cylinder radius="0.1" length="0.05"/>
+      </geometry>
+    </collision>
+    <visual>
+      <origin xyz="0 0 0" rpy="0 1.5707 1.5707"/>
+      <geometry>
+        <cylinder radius="0.1" length="0.05"/>
+      </geometry>
+    </visual>
+  </link>
+  <link name="right_wheel">
+    <inertial>
+      <mass value="5"/>
+      <origin xyz="0 0 0" rpy="0 1.5707 1.5707"/>
+      <inertia
+        ixx="0.1" ixy="0.0" ixz="0.0"
+        iyy="0.1" iyz="0.0"
+        izz="0.1"
+      />
+    </inertial>
+    <collision>
+      <origin xyz="0 0 0" rpy="0 1.5707 1.5707"/>
+      <geometry>
+        <cylinder radius="0.1" length="0.05"/>
+      </geometry>
+    </collision>
+    <visual>
+      <origin xyz="0 0 0" rpy="0 1.5707 1.5707"/>
+      <geometry>
+        <cylinder radius="0.1" length="0.05"/>
+      </geometry>
+    </visual>
+  </link>
 </robot>

Commit message: Added sensor and color

File: midge_ws/src/midge/urdf/midge.xacro (robot description, xacro)
@@ -1,4 +1,21 @@
 <?xml version='1.0'?>
+<!-- Robot Definition -->
 <robot name="midge" xmlns:xacro="http://www.ros.org/wiki/xacro">
+  <!-- Including Gazebo -->
+  <xacro:include filename="$(find midge)/urdf/midge.gazebo" />
+  <!-- Coloring all the parts -->
+  <gazebo reference='left_wheel'>
+    <material>Gazebo/Orange</material>
+  </gazebo>
+  <gazebo reference='right_wheel'>
+    <material>Gazebo/Orange</material>
+  </gazebo>
+  <gazebo reference='camera'>
+    <material>Gazebo/Red</material>
+  </gazebo>
+  <gazebo reference='chassis'>
+    <material>Gazebo/Black</material>
+  </gazebo>
+  <!-- Joint wheels and sensors -->
   <joint type="continuous" name="left_wheel_hinge">
     <origin xyz="0 0.30 0" rpy="0 0 0" />
@@ -17,4 +34,22 @@
     <dynamics damping="1.0" friction="1.0" />
   </joint>
+  <joint name="camera_joint" type="fixed">
+    <origin xyz="0.26 0 0" rpy="0 0 0" />
+    <parent link="chassis"/>
+    <child link="camera" />
+    <axis xyz="0 1 0"/>
+  </joint>
+  <joint name="hokuyo_joint" type="fixed">
+    <origin xyz="0.2 0 0.2" rpy="0 0 0" />
+    <parent link="chassis"/>
+    <child link="hokuyo" />
+    <axis xyz="0 1 0"/>
+  </joint>
+  <joint name="robot_footprint_joint" type="fixed">
+    <origin xyz="0 0 0" rpy="0 0 0" />
+    <parent link="robot_footprint"/>
+    <child link="chassis" />
+  </joint>
+  <!-- Chassis and sensor Definition -->
   <link name='chassis'>
     <pose>0 0 0.1 0 0 0</pose>
@@ -111,3 +146,51 @@
     </visual>
   </link>
+  <link name="camera">
+    <inertial>
+      <mass value="0.1"/>
+      <origin xyz="0 0 0" rpy="0 0 0"/>
+      <inertia
+        ixx="1e-6" ixy="0.0" ixz="0.0"
+        iyy="1e-6" iyz="0.0"
+        izz="1e-6"
+      />
+    </inertial>
+    <collision>
+      <origin xyz="0 0 0" rpy="0 0 0"/>
+      <geometry>
+        <box size="0.05 0.05 0.05"/>
+      </geometry>
+    </collision>
+    <visual>
+      <origin xyz="0 0 0" rpy="0 0 0"/>
+      <geometry>
+        <box size="0.05 0.05 0.05"/>
+      </geometry>
+    </visual>
+  </link>
+  <link name="hokuyo">
+      <inertial>
+        <mass value="1e-5"/>
+        <origin xyz="0 0 0" rpy="0 0 0"/>
+        <inertia
+          ixx="1e-6" ixy="0.0" ixz="0.0"
+          iyy="1e-6" iyz="0.0"
+          izz="1e-6"
+        />
+      </inertial>
+      <collision>
+        <origin xyz="0 0 0" rpy="0 0 0"/>
+        <geometry>
+          <box size="0.1 0.1 0.1"/>
+        </geometry>
+      </collision>
+      <visual>
+        <origin xyz="0 0 0" rpy="0 0 0"/>
+        <geometry>
+          <mesh filename="package://midge/meshes/hokuyo.dae"/>
+        </geometry>
+      </visual>
+    </link>
+  <link name="robot_footprint">
+  </link>
 </robot>

Commit message: Conclusione del progetto pronto per la presentazione

File: midge_ws/src/midge/urdf/midge.xacro (robot description, xacro)
@@ -19,5 +19,5 @@
   <!-- Joint wheels and sensors -->
   <joint type="continuous" name="left_wheel_hinge">
-    <origin xyz="0 0.30 0" rpy="0 0 0" />
+    <origin xyz="0 0.25 0" rpy="0 0 0" />
     <parent link="chassis"/>
     <child link="left_wheel" />
@@ -27,5 +27,5 @@
   </joint>
   <joint type="continuous" name="right_wheel_hinge">
-    <origin xyz="0 -0.30 0" rpy="0 0 0" />
+    <origin xyz="0 -0.25 0" rpy="0 0 0" />
     <parent link="chassis"/>
     <child link="right_wheel" />
